File: pcb/doorbell_pcb_v2/doorbell_pcb_v2/doorbell_pcb_v2.kicad_pcb (KiCad board)
At the start: 2 copper layers, 50 x 75 mm, 25 parts, among them J1 Screw_Terminal_01x02, J2 Screw_Terminal_01x02, J3 Conn_01x02_Pin, J4 Conn_01x03_Pin, SW1 MST22D18G2 125, U1 ACS712xLCTR-05B, U2 LM78M05_TO252

Commit message: PCB updates
Parts:
- removed the J3 at (170.0, 113.8)
- removed the R3 at (162.5, 109.5)
- J3: renamed from J4; footprint Connector_JST:JST_EH_B3B-EH-A_1x03_P2.50mm_Vertical -> Connector_PinHeader_2.54mm:PinHeader_1x03_P2.54mm_Vertical
- moved J3 28.3 mm to (141.8, 99.2), turned to 0 degrees
- moved TP1 8.95 mm to (146.8, 108.7)
- moved D2 6.96 mm to (141.6, 73.8)
- moved R3 3.80 mm to (138.6, 73.8), turned to -90 degrees
- moved D3 2.48 mm to (140.2, 78.6), turned to 180 degrees
- moved U3 2.15 mm to (149.4, 73.6)
- renumbered C5 to C4, C7 to C5, D3 to D2, D2 to D3, R4 to R3
Connections:
- J3 pad 2: /WS2812 -> +3.3V
- R3 pad 2: +5V Internal -> +5V
- U3 pad 10: /Ext Reset -> unconnected-(U3-GPIO_6-Pad10)
- U3 pad 18: /WS2812 -> unconnected-(U3-GPIO_21-Pad18)
Routing:
- net +5V Internal: track 94.4 -> 59.1 mm
- net /WS2812: track 33.8 -> 0.00 mm
- net /Ext Reset: track 28.7 -> 0.00 mm
- net GND: track 49.7 -> 24.9 mm, vias 11 -> 10
- net +3.3V: track 37.7 -> 27.2 mm
- net +5V: track 6.85 -> 10.9 mm
- net Net-(D2-A): track 2.23 -> 3.02 mm
- net /ADC Input: track 28.4 -> 28.9 mm
Other:
- board text added: "3V3"
- board text added: "5V"
- board text added: "Doorbell Ring Detector"
- board text added: "ESP32-C3 Zero"
- board text added: "GND"
- board text added: "OFF"
- board text added: "ON"
- board text added: "Vin (6-12V AC)"
- board text added: "Vout (6-12V AC)"
