File: pcb/doorbell_pcb_v2/doorbell_pcb_v2/doorbell_pcb_v2.kicad_sch (KiCad schematic)
At the start: 25 parts, among them J1 Screw_Terminal_01x02, J2 Screw_Terminal_01x02, J3 Conn_01x02_Pin, J4 Conn_01x03_Pin, SW1 MST22D18G2 125, U1 ACS712xLCTR-05B, U2 LM78M05_TO252

Commit message: PCB updates
Parts:
- removed J3: Conn_01x02_Pin, Connector_JST:JST_EH_B2B-EH-A_1x02_P2.50mm_Vertical, symbol Connector:Conn_01x02_Pin
- removed R3: 470R, Resistor_SMD:R_0805_2012Metric_Pad1.20x1.40mm_HandSolder, symbol Device:R
- added U4: DS18B20, Package_TO_SOT_THT:TO-92, symbol Sensor_Temperature:DS18B20
- J1, J2: LCSC (none) -> C474881
- J3: renamed from J4; footprint Connector_JST:JST_EH_B3B-EH-A_1x03_P2.50mm_Vertical -> Connector_PinHeader_2.54mm:PinHeader_1x03_P2.54mm_Vertical; now not fitted
- renumbered C5 to C4, C7 to C5, D3 to D2, D2 to D3, R4 to R3
Connections:
- net +3.3V: now also J3.2 (Pin_2)
- net +5V: now also R3.2
- net +5V Internal: no longer R3.2
- net Ext Reset: no longer names the net of U3.10 (GPIO_6)
- net WS2812: no longer names the net of U3.18 (GPIO_21)
- net WS2812: no longer J3.2 (Pin_2)
- no-connect marks 14 -> 16
Other:
- moved on the sheet: C5, D2, D3, R3
